Commit message: feat: modify robot xacro file

File: slam_project/urdf/new_robot.xacro (robot description, xacro)
@@ -80,6 +80,6 @@
       </geometry>
     </visual>
-    <visual name="box_visua">
-      <origin rpy="0.0 0 0.0" xyz="0.04 0 0.1"/>
+    <visual name="box_visual">
+      <origin rpy="0.0 0 0.0" xyz="0.04 0 0.12"/>
       <geometry>
         <box size=".08 .2 .1"/>
@@ -240,8 +240,8 @@
   </link>
   <gazebo reference="camera_link">
-    <material>Gazebo/Black</material>
+    <material>Gazebo/Green</material>
   </gazebo>
-  <joint type="continuous" name="camera_joint">
-    <origin xyz="0.18 0.0 0" rpy="0 0 0"/>
+  <joint type="fixed" name="camera_joint">
+    <origin xyz="0.04 0.0 0.2" rpy="0 0 0"/>
     <child link="camera_link"/>
     <parent link="chassis"/>
@@ -260,5 +260,5 @@
   </link>
   <joint name="camera_rgbd_joint" type="fixed">
-    <origin xyz="0 0.028 0" rpy="0 0 0" />
+    <origin xyz="0.04 0 0.26" rpy="0 0 0" />
     <parent link="camera_link" />
     <child link="camera_rgbd_frame" />
@@ -298,5 +298,5 @@
   </link>
   <joint type="continuous" name="hokuyo_joint">
-    <origin xyz="0.17 0.0 0.1" rpy="0 0 0"/>
+    <origin xyz="0.16 0.0 0.1" rpy="0 0 0"/>
     <child link="hokuyo"/>
     <parent link="chassis"/>

Commit message: feat: modify camera frame joint

File: slam_project/urdf/new_robot.xacro (robot description, xacro)
@@ -246,7 +246,4 @@
     <child link="camera_link"/>
     <parent link="chassis"/>
-    <axis xyz="0 1 0" rpy="0 0 0"/>
-    <limit effort="10000" velocity="1000"/>
-    <joint_properties damping="1.0" friction="1.0"/>
   </joint>
   <link name="camera_rgbd_frame">
@@ -260,5 +257,6 @@
   </link>
   <joint name="camera_rgbd_joint" type="fixed">
-    <origin xyz="0.04 0 0.26" rpy="0 0 0" />
+    <origin xyz="0.04 0 0.26" rpy="-1.57  0.0 -1.57" />
+       <!--origin xyz="0.04 0 0.26" rpy="0 0 0" /-->
     <parent link="camera_link" />
     <child link="camera_rgbd_frame" />
